Commit message: Update robot.urdf.xacro
Robot Model working well in gazebo - Also issue fixed of 2 root links error

File: src/robot_model_pkg/urdf/robot.urdf.xacro (robot description, xacro)
@@ -0,0 +1,219 @@
+<?xml version="1.0"?>
+<!-- Ensures xacro extension is being used -->
+<robot xmlns:xacro="http://www.ros.org/wiki/xacro" name="robot">
+    <!-- Setting up robot parameters -->
+  <xacro:property name="base_width" value="0.32"/>
+  <xacro:property name="base_len" value="0.32"/>
+  <xacro:property name="wheel_radius" value="0.07"/>
+  <xacro:property name="base_wheel_gap" value="0.007"/>
+  <xacro:property name="wheel_separation" value="0.30"/>
+  <xacro:property name="wheel_joint_offset" value="0.07"/>
+  <!-- Setting up caster wheel parameters  -->
+  <xacro:property name="caster_wheel_radius" value="${wheel_radius/2}"/>
+  <xacro:property name="caster_wheel_mass" value="0.002"/>
+  <xacro:property name="caster_wheel_joint_offset" value="-0.104"/>
+  <!-- Learning Point: Setting this paramters in beginning will avoid error of robot not being constructed properly and misaligned  -->
+  <!-- Includes plugin file created  -->
+  <xacro:include filename="$(find robot_model_pkg)/urdf/robot_gaz_drive.xacro"/>
+    <!-- Setting inertial for shapes so the model maintain common values  -->
+  <xacro:macro name="cylinder_inertia" params="m r h">
+    <inertial>
+      <mass value="${m}"/>
+      <inertia ixx="${m*(3*r*r+h*h)/12}" ixy = "0" ixz = "0" iyy="${m*(3*r*r+h*h)/12}" iyz = "0" izz="${m*r*r/2}"/>
+    </inertial>
+  </xacro:macro>
+  <xacro:macro name="box_inertia" params="m w h d">
+    <inertial>
+      <mass value="${m}"/>
+      <inertia ixx="${m / 12.0 * (d*d + h*h)}" ixy="0.0" ixz="0.0" iyy="${m / 12.0 * (w*w + h*h)}" iyz="0.0" izz="${m / 12.0 * (w*w + d*d)}"/>
+    </inertial>
+  </xacro:macro>
+  <xacro:macro name="sphere_inertia" params="m r">
+    <inertial>
+      <mass value="${m}"/>
+      <inertia ixx="${2.0*m*(r*r)/5.0}" ixy="0.0" ixz="0.0" iyy="${2.0*m*(r*r)/5.0}" iyz="0.0" izz="${2.0*m*(r*r)/5.0}"/>
+    </inertial>
+  </xacro:macro>
+  <!-- Learning Point: Set the inertial values for objective types in beginning to avoid the error of links being placed on different heights and not being attached  -->
+  <!-- Setting color values for robot properties -->
+  <material name="blue">
+    <color rgba="0 0 0.8 1"/>
+  </material>
+  <material name="black">
+    <color rgba="0 0 0 1"/>
+  </material>
+  <material name="white">
+    <color rgba="1 1 1 1"/>
+  </material>
+  <material name="red">
+    <color rgba="0.8 0.0 0.0 1.0"/>
+  </material>
+   <!-- Base object located under the robot chassis - To link all objects to construct the robot properly  -->  <link name="base">
+    <xacro:box_inertia m="10" w="0.001" h="0.001" d="0.001"/>
+    <visual>
+        <origin xyz="0 0 0" rpy="0 0 0" />
+        <geometry>
+            <box size="0.001 0.001 0.05" />
+        </geometry>
+    </visual>
+  </link>
+  <!-- Base_link is the main center box simulating the chassis  -->
+    <link name="base_link">
+    <xacro:box_inertia m="1" w="${base_len}" h="${base_width}" d="0.1"/>
+    <visual>
+      <geometry>
+        <box size="${base_len} ${base_width} 0.1"/>
+      </geometry>
+      <material name="black"/>
+    </visual>
+    <collision>
+      <geometry>
+        <box size="${base_len} ${base_width} 0.1"/>
+      </geometry>
+    </collision>
+  </link>
+  <!-- Learning Point: First draft of robot had a huge chassis box and caused an issue with navigating through the pillars. Therefore, above dimensions are quite small to be able to navigate easier -->
+  <!-- Connecting main base_link box with base to properly construct it   -->
+  <joint name="base_link_joint" type="fixed">
+    <origin xyz="0 0 ${wheel_radius + 0.005}" rpy="0 0 0" />
+    <parent link="base"/>
+    <child link="base_link" />
+  </joint>
+   <!-- Creating wheel links to move robot   -->
+  <xacro:macro name="wheel" params="prefix reflect">
+    <link name="${prefix}_wheel">
+      <visual>
+        <origin xyz="0 0 0" rpy="${pi/2} 0 0"/>
+        <geometry>
+          <cylinder radius="${wheel_radius}" length="0.01"/>
+        </geometry>
+        <material name="red"/>
+      </visual>
+      <collision>
+        <origin xyz="0 0 0" rpy="${pi/2} 0 0"/>
+        <geometry>
+          <cylinder radius="${wheel_radius}" length="0.01"/>
+        </geometry>
+      </collision>
+      <xacro:cylinder_inertia m="1" r="${wheel_radius}" h="0.01"/>
+    </link>
+    <!-- Connecting wheels with base_link box of robot -->
+    <joint name="${prefix}_wheel_joint" type="continuous">
+      <axis xyz="0 1 0" rpy="0 0 0" />
+      <parent link="base_link"/>
+      <child link="${prefix}_wheel"/>
+      <origin xyz="${wheel_joint_offset} ${((base_width/2)+base_wheel_gap)*reflect} -0.005" rpy="0 0 0"/>
+    </joint>
+  </xacro:macro>
+  <!-- Creating prefix and placing them opposite each other -->
+  <xacro:wheel prefix="left" reflect="1"/>
+  <xacro:wheel prefix="right" reflect="-1"/>
+  <!-- Learning Point: Setting the wheel with prefix names and parameters with prefix reflect allows the model to have perfectly aligned wheels as otherwise the wheels create don't work together to move the robot -->
+  <!-- Setting up caster wheel-->
+  <link name="caster_wheel">
+    <visual>
+      <origin xyz="0 0 0" rpy="0 0 0"/>
+      <geometry>
+        <sphere radius="${caster_wheel_radius}"/>
+      </geometry>
+      <material name="red"/>
+    </visual>
+    <collision>
+      <origin xyz="0 0 0" rpy="0 0 0"/>
+      <geometry>
+        <sphere radius="${caster_wheel_radius}"/>
+      </geometry>
+    </collision>
+    <xacro:sphere_inertia m="1" r="${caster_wheel_radius}"/>
+  </link>
+  <!-- Connecting caster wheel with base_link so it gets connected with robot -->
+  <joint name="caster_wheel_joint" type="continuous">
+    <axis xyz="0 1 0" rpy="0 0 0" />
+    <parent link="base_link"/>
+    <child link="caster_wheel"/>
+    <origin xyz="${caster_wheel_joint_offset} 0 -${caster_wheel_radius+0.005}" rpy="0 0 0"/>
+  </joint>
+<!-- Left guidance: used to represent left side of robot -->
+<link name="left_guide">
+  <xacro:box_inertia m="1" w="${base_len}" h="${base_width}" d="0.01"/>
+  <visual>
+    <geometry>
+      <box size="0.5 0.01 0.05"/>
+    </geometry>
+  <link name="left_guide">
+    <xacro:box_inertia m="1" w="${base_len}" h="${base_width}" d="0.01"/>
+    <visual>
+      <geometry>
+        <box size="0.5 0.01 0.05"/>
+      </geometry>
+      <material name="blue"/>
+    </visual>
+    <collision>
+      <geometry>
+        <box size="0.5 0.01 0.05"/>
+      </geometry>
+    </collision>
+  </link>
+  <!-- Left guidance: connecting link along with adding visual and collusion parameters  -->
+  <joint name="left_guide_joint" type="fixed">
+    <origin xyz="-0.2 0.5 0.0" rpy="0 0 0" />
+    <parent link="base"/>
+    <child link="left_guide" />
+  </joint>
+    <material name="blue"/>
+  </visual>
+  <collision>
+    <geometry>
+      <box size="0.5 0.01 0.05"/>
+    </geometry>
+  </collision>
+</link>
+<!-- Left guidance: connecting link to base-->
+<joint name="left_guide_joint" type="fixed">
+  <origin xyz="-0.2 0.15 0.06" rpy="0 0 0" />
+  <parent link="base"/>
+  <child link="left_guide" />
+</joint>
+<!--Right guidance: used to represent right side of robot -->
+<link name="right_guide">
+  <xacro:box_inertia m="1" w="${base_len}" h="${base_width}" d="0.01"/>
+  <visual>
+    <geometry>
+      <box size="0.5 0.01 0.05"/>
+    </geometry>
+  <link name="right_guide">
+    <xacro:box_inertia m="1" w="${base_len}" h="${base_width}" d="0.01"/>
+    <visual>
+      <geometry>
+        <box size="0.5 0.01 0.05"/>
+      </geometry>
+      <material name="blue"/>
+    </visual>
+    <collision>
+      <geometry>
+        <box size="0.5 0.01 0.05"/>
+      </geometry>
+    </collision>
+  </link>
+  <!-- Right guidance: connecting link along with adding visual and collusion parameters  -->
+  <joint name="right_guide_joint" type="fixed">
+    <origin xyz="-0.2 0.15 0.06" rpy="0 0 0" />
+    <parent link="base"/>
+    <child link="right_guide" />
+  </joint>
+    <material name="blue"/>
+  </visual>
+  <collision>
+    <geometry>
+      <box size="0.5 0.01 0.05"/>
+    </geometry>
+  </collision>
+</link>
+<!-- Right guidance: connecting link to base-->
+<joint name="right_guide_joint" type="fixed">
+  <origin xyz="-0.2 -0.15 0.06" rpy="0 0 0" />
+  <parent link="base"/>
+  <child link="right_guide" />
+</joint>
+<!-- Learning Point: Joints are for left and right guidance are set twice to properly set the connection to robot and to avoid the error about 2 root links conflicting each other  -->
+</robot>
